File: PicoClick/PicoClick.kicad_pcb (KiCad board)
At the start: 2 copper layers, 52 x 52 mm, 10 parts, among them J1 Conn_01x12_Socket, P1 CONN_8, P2 CONN_8, U1 W25Q128JVS

Commit message: fix SPI labels
Parts:
- A1: value RaspberryPi_Pico -> RaspberryPi_Pico2
- U1: value W25Q128JVS -> SST26F064B
Connections:
- net /G11_MOSI1 renamed /G11_SDO1
- net /G12_MISO1 renamed /G12_SDI1
- net /G16_MOSI0 renamed /G16_SDI0
- net /G19_MISO0 renamed /G19_SDO0
Other:
- board text added: "G16_SDI0"
- board text added: "G19_SDO0"
- board text removed: "G16_SDO0"
- board text removed: "G19_SDI0"
